Commit message: Created new URDF model of the robot

File: indigo_description/urdf/indigobot.urdf.xacro (robot description, xacro)
@@ -150,4 +150,28 @@
     <axis xyz="0 0 0" />
   </joint>
+<link name="caster_link">
+    <inertial>
+      <mass value="0.01"/>
+      <inertia ixx="1e-6" ixy="0" ixz="0" iyy="1e-6" iyz="0" izz="1e-6"/>
+    </inertial>
+    <visual>
+      <origin xyz="0 0 0" rpy="1.57 0 0" />
+      <geometry>
+        <cylinder radius="0.02" length="0.02"/>
+      </geometry>
+      <material name="silver"/>
+    </visual>
+    <collision>
+      <origin xyz="0 0 0" rpy="1.57 0 0" />
+      <geometry>
+        <cylinder radius="0.02" length="0.02"/>
+      </geometry>
+    </collision>
+</link>
+<joint name="caster_joint" type="fixed">
+    <origin xyz="0.057 0 -0.05" rpy="0 0 0"/>
+    <parent link="base_link"/>
+    <child link="caster_link"/>
+</joint>
   <material name="blue">
     <color rgba="0 0 1 1"/>

Commit message: Created new URDF model of the robot

File: indigo_description/urdf/indigobot.urdf.xacro (robot description, xacro)
@@ -50,5 +50,5 @@
         <mesh filename="package://indigo_description/meshes/wheel_right_link.STL" />
       </geometry>
-      <material name="blue"/>
+      <material name="black"/>
     </visual>
     <collision>
@@ -79,5 +79,5 @@
         <mesh filename="package://indigo_description/meshes/wheel_left_link.STL" />
       </geometry>
-      <material name="blue"/>
+      <material name="black"/>
     </visual>
     <collision>
@@ -107,5 +107,5 @@
         <mesh filename="package://indigo_description/meshes/imu_link.STL" />
       </geometry>
-      <material name="blue"/>
+      <material name="black"/>
     </visual>
     <collision>
@@ -160,5 +160,5 @@
         <cylinder radius="0.02" length="0.02"/>
       </geometry>
-      <material name="silver"/>
+      <material name="dark_grey"/>
     </visual>
     <collision>

Commit message: Updated and corrected URDF model

File: indigo_description/urdf/indigobot.urdf.xacro (robot description, xacro)
@@ -35,5 +35,5 @@
     <parent link="base_footprint"/>
     <child link="base_link" />
-    <origin xyz="0 0 0.033" rpy="0 0 0"/>
+    <origin xyz="0 0 0.072" rpy="0 0 0"/>
   </joint>
   <link name="wheel_right_link">

Commit message: updated URDF model

File: indigo_description/urdf/indigobot.urdf.xacro (robot description, xacro)
@@ -107,5 +107,5 @@
         <mesh filename="package://indigo_description/meshes/imu_link.STL" />
       </geometry>
-      <material name="black"/>
+      <material name="green"/>
     </visual>
     <collision>
@@ -186,3 +186,6 @@
     <color rgba="0.3 0.3 0.3 1"/>
   </material>
+  <material name="green">
+    <color rgba="0 1 0 1"/>
+  </material>
 </robot>

Commit message: added camera to URDF

File: indigo_description/urdf/indigobot.urdf.xacro (robot description, xacro)
@@ -174,4 +174,55 @@
     <child link="caster_link"/>
 </joint>
+<link
+    name="pt_camera_link">
+    <inertial>
+      <origin
+        xyz="0.00630730338217479 -7.90865732935165E-18 0.000950308188413934"
+        rpy="0 -1.5708 1.5708" />
+      <mass
+        value="0.00623651844028495" />
+      <inertia
+        ixx="5.11295942352593E-07"
+        ixy="3.46495200123478E-22"
+        ixz="-4.00917493406375E-08"
+        iyy="3.99078324787848E-07"
+        iyz="1.31404415819798E-22"
+        izz="4.02518684222241E-07" />
+    </inertial>
+    <visual>
+      <origin
+        xyz="0 0 0"
+        rpy="0 -1.5708 1.5708" />
+      <geometry>
+        <mesh
+          filename="package://indigo_description/meshes/camera_link.STL" />
+      </geometry>
+      <material
+        name="">
+        <color
+          rgba="0.627450980392157 0.627450980392157 0.627450980392157 1" />
+      </material>
+    </visual>
+    <collision>
+      <origin
+        xyz="0 0 0"
+        rpy="0 -1.5708 1.5708" />
+      <geometry>
+        <mesh
+          filename="package://indigo_description/meshes/camera_link.STL" />
+      </geometry>
+    </collision>
+  </link>
+  <joint
+    name="camera_joint"
+    type="fixed">
+    <origin
+      xyz="-0.07 0 0.05"
+      rpy="0 1.5708 3.14159" />
+    <parent
+      link="base_link" />
+    <child
+      link="pt_camera_link" />
+  </joint>
   <material name="blue">
     <color rgba="0 0 1 1"/>

Commit message: Added new LIDAR model to the robot

File: indigo_description/urdf/indigobot.urdf.xacro (robot description, xacro)
@@ -131,15 +131,13 @@
     </inertial>
     <visual>
-      <origin xyz="0 0 0" rpy="0 0 0" />
-      <geometry>
-        <mesh filename="package://indigo_description/meshes/laser_link.STL" />
+      <origin xyz="0 0 -0.045" rpy="0 0 3.14159" />
+      <geometry>
+        <mesh filename="package://indigo_description/meshes/ydlidar_x2l.stl" />
       </geometry>
       <material name="dark_grey"/>
     </visual>
     <collision>
-      <origin xyz="0 0 0" rpy="0 0 0" />
-      <geometry>
-        <mesh filename="package://indigo_description/meshes/laser_link.STL" />
-      </geometry>
+      <origin xyz="0 0 -0.0195" rpy="0 0 0"/>
+      <geometry><cylinder radius="0.035" length="0.051"/></geometry>
     </collision>
   </link>

Commit message: Actual wheel radius

File: indigo_description/urdf/indigobot.urdf.xacro (robot description, xacro)
@@ -55,5 +55,5 @@
       <origin xyz="0 -0.015 0" rpy="1.57 0 0" />
       <geometry>
-        <sphere radius="0.033"/>
+        <sphere radius="0.034"/>
       </geometry>
     </collision>
@@ -84,5 +84,5 @@
       <origin xyz="0 0.015 0" rpy="-1.57 0 0" />
       <geometry>
-        <sphere radius="0.033"/>
+        <sphere radius="0.034"/>
       </geometry>
     </collision>
